File: PMSX003-Breakout.sch (EAGLE design)
At the start: 3 parts

Commit message: Minor update
Other:
- note added: "PMS5003/7003 Breakout"
Changed lines of the file:
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@@
 <sheet>
 <plain>
+<text x="-66.04" y="58.42" size="1.778" layer="97" font="vector">PMS5003/7003 Breakout</text>
 </plain>
 <instances>
 <instance part="JP1" gate="A" x="-63.5" y="35.56" rot="R180"/>
 <instance part="U$1" gate="G$1" x="10.16" y="25.4"/>
-<instance part="U$2" gate="G$1" x="-15.24" y="10.16"/>
+<instance part="U$2" gate="G$1" x="-17.78" y="60.96"/>
 </instances>
 <busses>
